Commit message: 2018/7/24

File: my_robo_description/my_robo.urdf (robot description, URDF)
Before this commit: robot my_robo, 9 links, 8 joints
Links:
- removed link pico_flexx_depth_frame
- removed link pico_flexx_link
- removed link pico_flexx_link_optical_frame
Joints:
- removed joint pico_flexx_base_joint
- removed joint pico_flexx_depth_joint
- removed joint pico_flexx_joint
